File: gadgets/solderingChallenge/hardware/solderingChallenge.kicad_pcb (KiCad board)
At the start: 2 copper layers, 145 x 39 mm, 46 parts, among them J10 USB_A, J12 USB_A, J2 USB_A, J4 USB_A, J6 USB_A, J8 USB_A, U1 LM555xN, U2 LMC555xM, U3 LMC555xMM, U4 LMC555xMM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

Commit message: Rename smdChallenge to solderingChallenge
Other:
- board text added: "L1"
- board text added: "L2"
- board text added: "L3"
- board text added: "L4"
- board text added: "L5"
- board text added: "RoboticsBrno v1"
- board text added: "Soldering Challenge"
Changed lines of the file:
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@@
   (general
     (thickness 1.6)
-    (drawings 80)
+    (drawings 97)
     (tracks 308)
     (zones 0)
@@
     )
   )
+  (gr_text "RoboticsBrno\nv1" (at 92 75.5) (layer B.SilkS)
+    (effects (font (size 1 1) (thickness 0.15)) (justify mirror))
+  )
+  (gr_text L1 (at 90.5 93) (layer B.SilkS)
+    (effects (font (size 3 3) (thickness 0.7)) (justify mirror))
+  )
+  (gr_text L2 (at 117 93) (layer B.SilkS)
+    (effects (font (size 3 3) (thickness 0.7)) (justify mirror))
+  )
+  (gr_text "RoboticsBrno\nv1" (at 117 97) (layer B.SilkS)
+    (effects (font (size 1 1) (thickness 0.15)) (justify mirror))
+  )
+  (gr_text "Soldering\nChallenge\n" (at 117 88.5) (layer B.SilkS)
+    (effects (font (size 1.2 1.2) (thickness 0.2)) (justify mirror))
+  )
+  (gr_text L3 (at 142 94.5) (layer B.SilkS)
+    (effects (font (size 3 3) (thickness 0.7)) (justify mirror))
+  )
+  (gr_text "Soldering\nChallenge\n" (at 142 90) (layer B.SilkS)
+    (effects (font (size 1.2 1.2) (thickness 0.2)) (justify mirror))
+  )
+  (gr_text "RoboticsBrno\nv1" (at 142 98.5) (layer B.SilkS)
+    (effects (font (size 1 1) (thickness 0.15)) (justify mirror))
+  )
+  (gr_text "Soldering\nChallenge\n" (at 167 90) (layer B.SilkS)
+    (effects (font (size 1.2 1.2) (thickness 0.2)) (justify mirror))
+  )
+  (gr_text L4 (at 167 94.5) (layer B.SilkS)
+    (effects (font (size 3 3) (thickness 0.7)) (justify mirror))
+  )
+  (gr_text "RoboticsBrno\nv1" (at 167 98.5) (layer B.SilkS)
+    (effects (font (size 1 1) (thickness 0.15)) (justify mirror))
+  )
+  (gr_text L4 (at 192 94.5) (layer B.SilkS)
+    (effects (font (size 3 3) (thickness 0.7)) (justify mirror))
+  )
+  (gr_text "Soldering\nChallenge\n" (at 192 90) (layer B.SilkS)
+    (effects (font (size 1.2 1.2) (thickness 0.2)) (justify mirror))
+  )
+  (gr_text "RoboticsBrno\nv1" (at 192 98.5) (layer B.SilkS)
+    (effects (font (size 1 1) (thickness 0.15)) (justify mirror))
+  )
+  (gr_text "RoboticsBrno\nv1" (at 218 98.5) (layer B.SilkS)
+    (effects (font (size 1 1) (thickness 0.15)) (justify mirror))
+  )
+  (gr_text L5 (at 218 94.5) (layer B.SilkS)
+    (effects (font (size 3 3) (thickness 0.7)) (justify mirror))
+  )
+  (gr_text "Soldering\nChallenge\n" (at 218 90) (layer B.SilkS)
+    (effects (font (size 1.2 1.2) (thickness 0.2)) (justify mirror))
+  )
   (gr_text "THT Components" (at 91.9 74.9) (layer F.SilkS)
