File: gadgets/solderingChallenge/hardware/solderingChallenge.kicad_pcb (KiCad board)
At the start: 2 copper layers, 181.5 x 72 mm, 54 parts, among them J1 USB_A, J10 USB_A, J2 USB_A, J4 USB_A, J6 USB_A, J8 USB_A, U1 LM555xN, U2 LMC555xM, U3 LMC555xMM, U4 LMC555xMM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

Commit message: Rotate capacitor on L0
Parts:
- moved C12 5.00 mm to (60.0, 57.4), turned to 0 degrees
Routing:
- net Net-(C12-Pad1): track 53.3 -> 55.2 mm
Changed lines of the file:
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@@
   )
   (footprint "Capacitor_THT:C_Disc_D6.0mm_W2.5mm_P5.00mm" (layer "F.Cu")
-    (at 65 57.25 180)
+    (at 60 57.35)
     (descr "C, Disc series, Radial, pin pitch=5.00mm, , diameter*width=6*2.5mm^2, Capacitor, http://cdn-reichelt.de/documents/datenblatt/B300/DS_KERKO_TC.pdf")
     (tags "C Disc series Radial pin pitch 5.00mm  diameter 6mm width 2.5mm Capacitor")
@@
     (fp_line (start -0.5 1.25) (end 5.5 1.25) (layer "F.Fab") (width 0.1))
     (fp_line (start -0.5 -1.25) (end -0.5 1.25) (layer "F.Fab") (width 0.1))
-    (pad "1" thru_hole circle (at 0 0 180) (size 1.6 1.6) (drill 0.8) (layers *.Cu *.Mask)
+    (pad "1" thru_hole circle (at 0 0) (size 1.6 1.6) (drill 0.8) (layers *.Cu *.Mask)
       (net 38 "Net-(C12-Pad1)") (pintype "passive"))
-    (pad "2" thru_hole circle (at 5 0 180) (size 1.6 1.6) (drill 0.8) (layers *.Cu *.Mask)
+    (pad "2" thru_hole circle (at 5 0) (size 1.6 1.6) (drill 0.8) (layers *.Cu *.Mask)
       (net 37 "/Level 0 - THT/GND") (pintype "passive"))
     (model "${KICAD6_3DMODEL_DIR}/Capacitor_THT.3dshapes/C_Disc_D6.0mm_W2.5mm_P5.00mm.wrl"
@@
   (segment (start 69 90.75) (end 69 76.21) (width 1.5) (layer "F.Cu") (net 38))
   (segment (start 64.78 101.47) (end 62.24 104.01) (width 1.5) (layer "F.Cu") (net 38))
-  (segment (start 65 57.25) (end 65 72.21) (width 1.5) (layer "F.Cu") (net 38))
-  (segment (start 65 72.21) (end 65.04 72.25) (width 1.5) (layer "F.Cu") (net 38))
+  (segment (start 60 67.21) (end 60 57.35) (width 1.5) (layer "F.Cu") (net 38))
   (segment (start 64.78 98.43) (end 64.78 101.47) (width 1.5) (layer "F.Cu") (net 38))
   (segment (start 62.24 104.01) (end 62.24 106.05) (width 1.5) (layer "F.Cu") (net 38))
   (segment (start 64.78 94.97) (end 69 90.75) (width 1.5) (layer "F.Cu") (net 38))
+  (segment (start 65.04 72.25) (end 60 67.21) (width 1.5) (layer "F.Cu") (net 38))
   (segment (start 82.5 62.29) (end 82.5 78.5) (width 1.5) (layer "F.Cu") (net 39))
   (segment (start 85 99.370946) (end 85 101.5) (width 1.5) (layer "F.Cu") (net 40))
