File: gadgets/solderingChallenge/hardware/level1-THT.sch (KiCad schematic (older format))
At the start: 8 parts, among them J2 USB_A, U1 LM555xN

Commit message: Last minute touches
Parts:
- J2: symbol Connector:USB_A -> solderingChallenge-rescue:USB_A-Connector
Changed lines of the file:
@@
 $Descr A4 11693 8268
 encoding utf-8
-Sheet 2 7
+Sheet 2 6
 Title ""
 Date ""
@@
 Connection ~ 5300 4450
 $Comp
-L Connector:USB_A J?
+L solderingChallenge-rescue:USB_A-Connector J?
 U 1 1 600F9A85
 P 4450 3450
