File: gadgets/solderingChallenge/hardware/level2-1206.sch (KiCad schematic (older format))
At the start: 8 parts, among them J4 USB_A, U2 LMC555xM

Commit message: Last minute touches
Parts:
- J4: symbol Connector:USB_A -> solderingChallenge-rescue:USB_A-Connector
Changed lines of the file:
@@
 $Descr A4 11693 8268
 encoding utf-8
-Sheet 3 7
+Sheet 3 6
 Title ""
 Date ""
@@
 Connection ~ 5000 4400
 $Comp
-L Connector:USB_A J?
+L solderingChallenge-rescue:USB_A-Connector J?
 U 1 1 600FC9C2
 P 4150 3400
