File: gadgets/solderingChallenge/hardware/level3-0603.sch (KiCad schematic (older format))
At the start: 8 parts, among them J6 USB_A, U3 LMC555xMM

Commit message: Last minute touches
Parts:
- J6: symbol Connector:USB_A -> solderingChallenge-rescue:USB_A-Connector
Changed lines of the file:
@@
 $Descr A4 11693 8268
 encoding utf-8
-Sheet 4 7
+Sheet 4 6
 Title ""
 Date ""
@@
 Connection ~ 5300 4350
 $Comp
-L Connector:USB_A J?
+L solderingChallenge-rescue:USB_A-Connector J?
 U 1 1 600FE73B
 P 4450 3350
