File: gadgets/solderingChallenge/hardware/level4-0402.sch (KiCad schematic (older format))
At the start: 8 parts, among them J8 USB_A, U4 LMC555xMM

Commit message: Last minute touches
Parts:
- J8: symbol Connector:USB_A -> solderingChallenge-rescue:USB_A-Connector
Changed lines of the file:
@@
 $Descr A4 11693 8268
 encoding utf-8
-Sheet 5 7
+Sheet 5 6
 Title ""
 Date ""
@@
 Connection ~ 5150 4550
 $Comp
-L Connector:USB_A J?
+L solderingChallenge-rescue:USB_A-Connector J?
 U 1 1 601033CC
 P 4300 3550
