File: gadgets/solderingChallenge/hardware/level5-0201.sch (KiCad schematic (older format))
At the start: 8 parts, among them J10 USB_A, U5 LMC555xTP

Commit message: Last minute touches
Parts:
- J10: symbol Connector:USB_A -> solderingChallenge-rescue:USB_A-Connector
Changed lines of the file:
@@
 $Descr A4 11693 8268
 encoding utf-8
-Sheet 6 7
+Sheet 6 6
 Title ""
 Date ""
@@
 Connection ~ 5300 4250
 $Comp
-L Connector:USB_A J?
+L solderingChallenge-rescue:USB_A-Connector J?
 U 1 1 6010069B
 P 4450 3250
