File: gadgets/solderingChallenge/hardware/solderingChallenge.sch (KiCad schematic (older format))
At the start: 0 parts

Commit message: Last minute touches
Changed lines of the file:
@@
 $Descr A4 11693 8268
 encoding utf-8
-Sheet 1 7
+Sheet 1 6
 Title ""
 Date ""
@@
 F1 "level5-0201.sch" 50
 $EndSheet
-$Sheet
-S 6450 4750 1700 950
-U 60142645
-F0 "Level 4 alternative - 0402" 50
-F1 "leve4-alt-0402.sch" 50
-$EndSheet
 $EndSCHEMATC
