File: gadgets/electronicDie/hardware/electronicDie.brd (EAGLE design)
At the start: 43.2 x 69.8 mm, 32 parts, among them IC1 CD4029N, IC2 NE555N, T1 BC327, T2 BC337, X1 USBPCB

Commit message: Add NC symbol to USB data pins
Connections:
- new net N$23: X1.USB_M
- new net N$24: X1.USB_P
Changed lines of the file:
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@@
 <wire x1="19.685" y1="59.69" x2="18.88" y2="58.885" width="0.508" layer="1"/>
+</signal>
+<signal name="N$23">
+<contactref element="X1" pad="USB_M"/>
+</signal>
+<signal name="N$24">
+<contactref element="X1" pad="USB_P"/>
 </signal>
 </signals>
