File: gadgets/usbPad/hardware/usbPad.kicad_pcb (KiCad board)
At the start: 2 copper layers, 12 x 12 mm, 1 part

Commit message: Change Helceletka branding
Parts:
- moved svg2mod 0.50 mm to (150.0, 91.5)
Other:
- board text added: "DDM Helceletka"
- board text removed: "DDM Helceletova"
