File: gadgets/electronicDie/hardware/v1.1/electronicDie.brd (EAGLE design)
At the start: 48.3 x 90.2 mm, 30 parts, among them IC1 CD4029N, IC2 NE555N, T1 BC557B, T2 BC547B, X1 USBPCB

Commit message: ElectronicDie v1.2: more resistant to assembly errors - resistors with same value grouped together - diodes grouped together - larger spaces between parts - 2k2 resistor replaced with 2 × 1k (so only 3 types of resistors left: 1k, 10k and 4M7) - added parts value to silkscreen - URL in silkscreen changed from robotikabrno.cz to robotickytabor.cz - changed year of Robocamp to 2022 (but 2021 remains in repo URL) - added silkscreen label for engraving owner name
Other:
- board text added: "JLCJLCJLCJLC"
Changed lines of the file:
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@@
 <setting verticaltext="up"/>
 </settings>
-<grid distance="50" unitdist="mil" unit="mil" style="lines" multiple="1" display="no" altdistance="25" altunitdist="mil" altunit="mil"/>
+<grid distance="50" unitdist="mil" unit="mil" style="lines" multiple="1" display="yes" altdistance="25" altunitdist="mil" altunit="mil"/>
 <layers>
 <layer number="1" name="Top" color="4" fill="1" visible="yes" active="yes"/>
@@
 <layer number="45" name="Holes" color="7" fill="1" visible="yes" active="yes"/>
 <layer number="46" name="Milling" color="3" fill="1" visible="no" active="yes"/>
-<layer number="47" name="Measures" color="7" fill="1" visible="no" active="yes"/>
+<layer number="47" name="Measures" color="7" fill="1" visible="yes" active="yes"/>
 <layer number="48" name="Document" color="7" fill="1" visible="yes" active="yes"/>
 <layer number="49" name="Reference" color="7" fill="1" visible="yes" active="yes"/>
@@
 <dimension x1="40.64" y1="24.13" x2="40.64" y2="40.64" x3="58.42" y3="32.385" textsize="1.27" textratio="16" layer="47" dtype="horizontal"/>
 <dimension x1="24.13" y1="13.97" x2="36.83" y2="32.385" x3="53.34" y3="23.1775" textsize="1.27" textratio="16" layer="47" dtype="vertical"/>
+<text x="24.13" y="78.74" size="0.8128" layer="102" font="vector" ratio="16" rot="SMR0" align="bottom-center">JLCJLCJLCJLC</text>
 <dimension x1="24.13" y1="24.13" x2="40.64" y2="24.13" x3="32.385" y3="-6.35" textsize="1.27" layer="47"/>
 <dimension x1="40.64" y1="7.62" x2="40.64" y2="40.64" x3="66.04" y3="24.13" textsize="1.27" layer="47"/>
